File: hw-trv/kicad/trv.kicad_pcb (KiCad board)
At the start: 2 copper layers, 100 x 100 mm, 269 parts, among them IC1 RFFC2071TR13, IC2 MHT2012NT1, J1 VCC+PTT, J2 TRX, J3 SWD ISP, J4 RX_OUT / 25M_REF, J5 LNB, J6 TX, Q1 BC848, Q2 BC847C, Q3 BSS84P, Q4 MMBT3904, Q5 MJE122, Q6 BSS84P, SW1 SW_DIP_x03, T1 ETC1.6-4-2-3TR, T2 MABACT0039, T3 MABACT0039, T4 ETC1.6-4-2-3TR, U1 STM32L011D4P6TR, U10 MAX20457ATIF/VY+, U11 L78L09ACUTR, U2 LM321, U3 SKY66292-11, U4 74LVC2G17, U5 TPS73633DBVRG4, U6 LP2985-18DBVR, U7 MIC5219-3.0YMM, U8 TLV74130PDBVR, U9 TLV74130PDBVR, X1 TA1862A, X2 TA1862A, Y1 LFTVXO076346 25MHz

Commit message: release: 1.0
Parts:
- removed ? (x5): , 
- removed C103, C42, C44: 100n, Capacitor_SMD:C_0603_1608Metric_Pad1.08x0.95mm_HandSolder
- removed C43: 0, Capacitor_SMD:C_0603_1608Metric_Pad1.08x0.95mm_HandSolder
- removed C45: 1, Capacitor_SMD:C_0402_1005Metric
- removed JP5: SolderJumper_2_Open, Jumper:SolderJumper-2_P1.3mm_Bridged_RoundedPad1.0x1.5mm
- removed Q1: BC848, Package_TO_SOT_SMD:SOT-23
- removed Q2: BC847C, Package_TO_SOT_SMD:SOT-23
- removed Q4: MMBT3904, Package_TO_SOT_SMD:SOT-23
- removed Q5: MJE122, Connector_PinHeader_1.27mm:PinHeader_1x03_P1.27mm_Vertical
- removed R23: 220, Resistor_SMD:R_0603_1608Metric_Pad0.98x0.95mm_HandSolder
- removed R24: 6.8k, Resistor_SMD:R_0603_1608Metric_Pad0.98x0.95mm_HandSolder
- removed R25: 15k, Resistor_SMD:R_0603_1608Metric_Pad0.98x0.95mm_HandSolder
- removed R26: 10k, Resistor_SMD:R_0603_1608Metric_Pad0.98x0.95mm_HandSolder
- removed R27: 2.7k, Resistor_SMD:R_0603_1608Metric_Pad0.98x0.95mm_HandSolder
- removed R30, R32: 16, Resistor_SMD:R_0603_1608Metric_Pad0.98x0.95mm_HandSolder
- removed R33: 100k, Resistor_SMD:R_0603_1608Metric_Pad0.98x0.95mm_HandSolder
- removed R36: 1k, Resistor_SMD:R_0603_1608Metric_Pad0.98x0.95mm_HandSolder
- removed R37: 330, Resistor_SMD:R_0603_1608Metric_Pad0.98x0.95mm_HandSolder
- removed R38: 3, Resistor_SMD:R_1812_4532Metric
- removed the REF** at (226.2, 101.0)
- removed the REF** at (226.2, 137.0)
- removed the REF** at (131.8, 150.2)
- removed the REF** at (131.8, 152.4)
- removed the REF** at (128.5, 151.1)
- removed T3: MABACT0039, Library:MABACT0039_MCM
- removed TH1: 10k, Connector_PinHeader_1.27mm:PinHeader_1x02_P1.27mm_Vertical
- removed U2: LM321, Package_TO_SOT_SMD:SOT-23-5
- removed X1, X2: TA1862A, Filter:Filter_SAW_Epcos_DCC6C_3x3mm
- removed rx: RX, 
- added C114: 33, Capacitor_SMD:C_0603_1608Metric_Pad1.08x0.95mm_HandSolder, F.Cu at (214.7, 151.3)
- added C115: 1n, Capacitor_SMD:C_0603_1608Metric_Pad1.08x0.95mm_HandSolder, F.Cu at (238.5, 174.9)
- added D9: BAT54WS, Diode_SMD:D_SOD-323F, F.Cu at (164.6, 174.8)
- added FL4: B39242B7520P810, Filter:SMD5_SAW-B7520_QUA, F.Cu at (204.5, 146.0)
- added FL5: B39242B7520P810, Filter:SMD5_SAW-B7520_QUA, F.Cu at (201.9, 146.2)
- added HY1: PD0409J5050S2HF, Wilkinson_splitter:PD0409J5050S2HF, F.Cu at (212.2, 163.1)
- added L13: 390n, Inductor_SMD:L_Cenker_CKCS252012, F.Cu at (231.1, 148.2)
- added Q7: BC847BDW1, Package_TO_SOT_SMD:SOT-363_SC-70-6, F.Cu at (233.0, 159.5)
- added REF**: TestPoint_Pad_2.0x2.0mm, TestPoint:TestPoint_Pad_2.0x2.0mm, F.Cu at (228.7, 185.8)
- added REF**: TestPoint_Pad_2.0x2.0mm, TestPoint:TestPoint_Pad_2.0x2.0mm, F.Cu at (213.5, 182.7)
- added REF**: TestPoint_Pad_2.0x2.0mm, TestPoint:TestPoint_Pad_2.0x2.0mm, F.Cu at (231.8, 185.8)
- added REF**: TestPoint_Pad_2.0x2.0mm, TestPoint:TestPoint_Pad_2.0x2.0mm, F.Cu at (219.6, 182.7)
- added REF**: TestPoint_Pad_2.0x2.0mm, TestPoint:TestPoint_Pad_2.0x2.0mm, F.Cu at (216.5, 185.8)
- added REF**: TestPoint_Pad_2.0x2.0mm, TestPoint:TestPoint_Pad_2.0x2.0mm, F.Cu at (228.7, 182.7)
- added REF**: TestPoint_Pad_1.0x1.0mm, TestPoint:TestPoint_Pad_1.0x1.0mm, F.Cu at (162.0, 176.5)
- added REF**: TestPoint_Pad_2.0x2.0mm, TestPoint:TestPoint_Pad_2.0x2.0mm, F.Cu at (222.6, 182.7)
- added REF**: MountingHole_3.5mm, MountingHole:MountingHole_3.5mm, F.Cu at (226.2, 101.0)
- added REF**: TestPoint_Pad_2.0x2.0mm, TestPoint:TestPoint_Pad_2.0x2.0mm, F.Cu at (213.5, 185.8)
- added REF**: TestPoint_Pad_2.0x2.0mm, TestPoint:TestPoint_Pad_2.0x2.0mm, F.Cu at (219.6, 185.8)
- added REF**: TestPoint_Pad_2.0x2.0mm, TestPoint:TestPoint_Pad_2.0x2.0mm, F.Cu at (216.5, 182.7)
- added REF**: TestPoint_Pad_2.0x2.0mm, TestPoint:TestPoint_Pad_2.0x2.0mm, F.Cu at (225.7, 182.7)
- added REF**: TestPoint_Pad_2.0x2.0mm, TestPoint:TestPoint_Pad_2.0x2.0mm, F.Cu at (231.8, 182.7)
- added REF**: TestPoint_Pad_2.0x2.0mm, TestPoint:TestPoint_Pad_2.0x2.0mm, F.Cu at (222.6, 185.8)
- added REF**: MountingHole_3.5mm, MountingHole:MountingHole_3.5mm, F.Cu at (226.2, 137.0)
- added REF**: TestPoint_Pad_2.0x2.0mm, TestPoint:TestPoint_Pad_2.0x2.0mm, F.Cu at (225.7, 185.8)
- added REF**: TestPoint_Pad_2.0x2.0mm, TestPoint:TestPoint_Pad_2.0x2.0mm, F.Cu at (234.8, 182.7)
- added REF**: TestPoint_Pad_2.0x2.0mm, TestPoint:TestPoint_Pad_2.0x2.0mm, F.Cu at (234.8, 185.8)
- C104: value 2.2u -> 4.7u
- C110, C96, C99: footprint Capacitor_SMD:C_0805_2012Metric_Pad1.18x1.45mm_HandSolder -> Capacitor_SMD:C_1206_3216Metric
- C112: footprint Capacitor_SMD:C_0805_2012Metric_Pad1.18x1.45mm_HandSolder -> Capacitor_SMD:C_1206_3216Metric_Pad1.33x1.80mm_HandSolder
- C29: value 1n -> 15
- C3, C4: footprint Capacitor_SMD:C_0805_2012Metric_Pad1.18x1.45mm_HandSolder -> Capacitor_SMD:C_0603_1608Metric_Pad1.08x0.95mm_HandSolder
- C36: value 100 -> 470
- C37: value 100 -> 0
- C41: value 100n -> 0
- C51: value 1.8 -> 2.2
- C55: value 100n -> 1n
- C56: value 12 -> 27
- C59: value 4.7 -> 5.6
- C7: value 100 * -> 100
- C79: value 2.2u -> 4.7u; footprint Capacitor_SMD:C_0603_1608Metric_Pad1.08x0.95mm_HandSolder -> Capacitor_Tantalum_SMD:CP_EIA-3528-21_Kemet-B_HandSolder
- C88: value 1.6 -> 2.2 / 1.6
- D3: value BAT54 -> BAT54WS; footprint Diode_SMD:D_SOD-123 -> Diode_SMD:D_SOD-323F
- F1: value 1.85A -> 1.5A
- FL2: value TA0532A -> F5QA737M5M2QN-J; footprint Filter:Filter_SAW_Epcos_DCC6C_3x3mm -> Filter:SMD5_SAW-B7520_QUA
- FL3: value TA0532A -> FAR-F5KY-740M00-B4UR-Z; footprint Filter:Filter_SAW_Epcos_DCC6C_3x3mm -> FAR-F5KY:FAR-F5KY
- J2, J4: footprint Connector_Coaxial:SMA_Wurth_60312102114405_Vertical -> Connector_Coaxial:SMA_Amphenol_132289_EdgeMount
- J5: footprint Connector_Coaxial:SMA_Wurth_60312102114405_Vertical -> F_conn:222131
- L10: value 1u -> 820n; footprint Inductor_SMD:L_0603_1608Metric_Pad1.05x0.95mm_HandSolder -> Inductor_SMD:L_1008_2520Metric_Pad1.43x2.20mm_HandSolder
- L12: footprint Inductor_SMD:L_Walsin_WLFM201209x -> Inductor_SMD:L_0603_1608Metric_Pad1.05x0.95mm_HandSolder
- L16: footprint Fuse:Fuse_1812_4532Metric_Pad1.30x3.40mm_HandSolder -> Inductor_SMD:L_1812_4532Metric_Pad1.30x3.40mm_HandSolder
- L2: value 0.22u -> 1u; footprint Inductor_SMD:L_0805_2012Metric_Pad1.05x1.20mm_HandSolder -> Inductor_SMD:L_1008_2520Metric_Pad1.43x2.20mm_HandSolder
- L3: value 1u -> 4.7u
- L4, L5: footprint Inductor_SMD:L_0402_1005Metric -> Inductor_SMD:L_0603_1608Metric_Pad1.05x0.95mm_HandSolder
- L6: value BK1608HM102TL -> 742792693
- L7: value 120n -> 68n
- L8: value 10n -> 12n
- L9: value 180nH -> 100n
- R1, R3: value 4k7 -> 4.7k
- R12: value 56/5W -> 56; footprint Resistor_THT:R_Axial_DIN0614_L14.3mm_D5.7mm_P15.24mm_Horizontal -> res_3550:RES_3550_TEC
- R15: value 0 -> 47k
- R28: value 16 -> 100
- R41, R43: value 270 -> 910
- R42: value 18 -> 5.6
- R51: value 10k -> 22k
- R56: value 560k -> 121.2K
- R57: value 47k -> 10k
- RV2: footprint Potentiometer_SMD:Potentiometer_Bourns_3269W_Vertical -> Potentiometer_SMD:Potentiometer_Bourns_3314J_Vertical
- T1: value ETC1.6-4-2-3TR -> TC4-19+
- U3: value SKY66292-11 -> SKY66312-11
- moved R20 83.1 mm to (204.0, 100.3), turned to 90 degrees
- moved R18 55.6 mm to (214.6, 141.8)
- moved R48 52.3 mm to (182.5, 150.8)
- moved C64 49.0 mm to (183.7, 154.2), turned to 0 degrees
- moved Q6 45.7 mm to (183.5, 147.2)
- moved C41 32.3 mm to (232.6, 166.2), turned to 0 degrees
- moved J4 27.8 mm to (247.7, 183.9), turned to 0 degrees
- moved C37 25.4 mm to (230.3, 152.0), turned to 0 degrees
- moved C51 23.9 mm to (220.8, 164.0)
- moved C36 23.5 mm to (230.9, 150.5), turned to 0 degrees
- moved C48 23.5 mm to (217.1, 168.5), turned to 0 degrees
- moved L8 23.2 mm to (220.8, 166.4), turned to 45 degrees
- moved C59 23.0 mm to (224.2, 165.2)
- moved FL2 22.3 mm to (218.1, 164.0), turned to -90 degrees
- moved 9V 20.5 mm to (184.2, 143.9)
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Connections:
- net +2V8 renamed +3V/uC
- net Net-(J3-Pin_3) renamed //RST
- C36 pad 2: Net-(JP2-C) -> GND
- C41 pad 1: +9V -> GND
- C41 pad 2: GND -> Net-(C41-Pad2)
- C51 pad 2: Net-(X2-OUT) -> Net-(FL2-IN)
- C74 pad 2: VBUS -> Net-(IC2-VDS1)
- C83 pad 1: GND -> VBUS
- C83 pad 2: VBUS -> GND
- C87 pad 2: VBUS -> Net-(IC2-VDS2_2)
- FL2 pad 1: GND -> Net-(FL2-IN)
- FL2 pad 2: Net-(FL2-IN) -> GND
- FL2 pad 4: GND -> Net-(FL2-OUT)
- FL2 pad 5: Net-(FL2-OUT) -> GND
- FL3 pad 1: GND -> Net-(FL3-IN)
- FL3 pad 2: Net-(FL2-OUT) -> GND
- FL3 pad 3: GND -> Net-(IC1A-MIX1_IPP)
- FL3 pad 4: GND -> Net-(IC1A-MIX1_IPN)
- FL3 pad 5: Net-(FL3-OUT) -> GND
- IC2 pad 10: VBUS -> Net-(IC2-VDS1)
- IC2 pad 11: VBUS -> Net-(IC2-VDS1)
- IC2 pad 16: VBUS -> Net-(IC2-VDS2_2)
- IC2 pad 17: VBUS -> Net-(IC2-VDS2_2)
- IC2 pad 18: VBUS -> Net-(IC2-VDS2_2)
- IC2 pad 9: VBUS -> Net-(IC2-VDS1)
- J3 pad 6: unconnected-(J3-Pin_6-Pad6) -> /BOOT
- JP1 pad 3: Net-(JP1-B) -> Net-(HY1-OUTPUT_1)
- JP2 pad 2: Net-(JP2-C) -> Net-(FL3-IN)
- JP2 pad 3: Net-(JP2-B) -> Net-(HY1-OUTPUT_2)
- JP4 pad 2: Net-(JP4-C) -> Net-(FL2-OUT)
- JP6 pad 1: Net-(JP6-A) -> Net-(JP1-A)
- JP6 pad 3: Net-(JP1-A) -> Net-(JP6-B)
- L10 pad 2: Net-(L10-Pad2) -> Net-(C41-Pad2)
- L11 pad 1: Net-(L10-Pad2) -> Net-(C41-Pad2)
- L2 pad 1: Net-(C7-Pad1) -> Net-(C37-Pad1)
- L2 pad 2: Net-(L2-Pad2) -> Net-(C36-Pad1)
- L3 pad 1: Net-(D4-A) -> Net-(C37-Pad1)
- L3 pad 2: Net-(L2-Pad2) -> Net-(C7-Pad1)
- L7 pad 1: Net-(JP6-A) -> Net-(JP6-B)
- L9 pad 2: Net-(JP7-A) -> Net-(C115-Pad2)
- R15 pad 1: /RFFC_SDATA -> GND
- R15 pad 2: Net-(U1-PA7) -> /BOOT
- R18 pad 1: /RFFC_SCLK -> Net-(R18-Pad1)
- R18 pad 2: Net-(U1-PA9) -> Net-(Q6-D)
- R20 pad 1: /RFFC_ENX -> Net-(Q6-D)
- R20 pad 2: Net-(U1-PA10) -> Net-(R20-Pad2)
- R28 pad 1: Net-(JP2-B) -> Net-(HY1-OUTPUT_1)
- R28 pad 2: Net-(R28-Pad2) -> Net-(HY1-OUTPUT_2)
- R31 pad 2: Net-(FL2-IN) -> Net-(FL4-IN)
- R35 pad 2: Net-(FL2-IN) -> Net-(FL4-IN)
- R41 pad 2: Net-(FL3-OUT) -> Net-(FL5-OUT)
- R42 pad 1: Net-(FL3-OUT) -> Net-(FL5-OUT)
- RV3 pad 1: Net-(Q6-D) -> Net-(R18-Pad1)
- RV4 pad 3: Net-(Q6-D) -> Net-(R20-Pad2)
- U1 pad 1: unconnected-(U1-PB9-Pad1) -> /BOOT
- U1 pad 11: Net-(U1-PA9) -> /RFFC_SCLK
- U1 pad 12: Net-(U1-PA10) -> /RFFC_ENX
- U1 pad 8: Net-(U1-PA7) -> /RFFC_SDATA
Routing:
- net +9V: track 83.1 -> 12.9 mm, vias 4 -> 0
- net GND: track 44.1 -> 112.6 mm, vias 1348 -> 1937
- net Net-(JP5-A): track 38.3 -> 0.00 mm, vias 3 -> 0
- net +5V: track 165.3 -> 129.7 mm, vias 11 -> 10
- net Net-(C115-Pad2): track 0.00 -> 34.8 mm, vias 0 -> 5
- net Net-(JP1-C): track 2.22 -> 32.1 mm
- net //PA_ENABLE: track 173.2 -> 198.3 mm, vias 9 -> 7
- net /LNB_REF: track 29.0 -> 5.94 mm, vias 2 -> 0
- net Net-(D4-K): track 33.5 -> 10.9 mm, vias 1 -> 0
- net Net-(JP7-A): track 25.0 -> 4.25 mm, vias 4 -> 0
- net /BOOT: track 0.00 -> 18.9 mm
- net Net-(HY1-OUTPUT_1): track 0.00 -> 16.9 mm
- net Net-(X2-OUT): track 16.2 -> 0.00 mm
- net Net-(IC2-VDS1): track 0.00 -> 13.9 mm
- net Net-(D8-A): track 2.36 -> 16.1 mm, vias 0 -> 2
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- added copper zone on B.Cu, net VBUS
Other:
- outline, holes or cut-outs redrawn
- board text added: "C108"
- board text added: "MHT2012N"
- board text added: "PD0409J5050S2HF"
- board text added: "RFFC2071"
- board text added: "rev 1.0 SQ5NRY designed in Poland"
- board text added: "x"
- board text removed: "rev 0.2 SQ5NRY Made in Poland"
