File: hw-trv/kicad/trv.kicad_sch (KiCad schematic)
At the start: 251 parts, among them IC1 RFFC2071TR13, IC2 MHT2012NT1, J1 VCC+PTT, J2 TRX, J3 SWD ISP, J4 RX_OUT / 25M_REF, J5 LNB, J6 TX, Q1 BC848, Q2 BC848B, Q3 BSS84P, Q4 MMBT3904, Q5 MJE122, Q6 BSS84P, SW1 SW_DIP_x03, T1 TC4-19+, T2 MABACT0039, T3 MABACT0039, T4 ETC1.6-4-2-3TR, U1 STM32L011D4P6TR, U10 MAX20457ATIF/VY+, U11 L78L09ACUTR, U13 PD0409J5050S2HF, U2 LM321, U3 SKY66292-11, U4 74LVC2G17, U5 TPS73633DBVRG4, U6 LP2985-18DBVR, U7 MIC5219-3.0YMM, U8 TLV74130PDBVR, U9 TLV74130PDBVR, X1 TA1862A, X2 TA1862A, Y1 LFTVXO076346 25MHz

Commit message: release: 1.0
Parts:
- removed C103, C42, C44: 100n, Capacitor_SMD:C_0603_1608Metric_Pad1.08x0.95mm_HandSolder, symbol Device:C_Small
- removed C43: 0, Capacitor_SMD:C_0603_1608Metric_Pad1.08x0.95mm_HandSolder, symbol Device:C_Small
- removed C45: 0.8, Capacitor_SMD:C_0402_1005Metric, symbol Device:C_Small
- removed FL2, FL3: TA0532A, Filter:Filter_SAW_Epcos_DCC6C_3x3mm, symbol RF_Filter:BFCN-2450
- removed JP8, JP9: SolderJumper_2_Open, Jumper:SolderJumper-2_P1.3mm_Bridged_RoundedPad1.0x1.5mm, symbol Jumper:SolderJumper_2_Open
- removed L22: 15n, Inductor_SMD:L_Coilcraft_0805HQ_2012Metric, symbol Device:L
- removed Q1: BC848, Package_TO_SOT_SMD:SOT-23, symbol Transistor_BJT:BC848
- removed Q2: BC848B, Package_TO_SOT_SMD:SOT-23, symbol Transistor_BJT:BC848
- removed Q4: MMBT3904, Package_TO_SOT_SMD:SOT-23, symbol Transistor_BJT:MMBT3904
- removed Q5: MJE122, Connector_PinHeader_1.27mm:PinHeader_1x03_P1.27mm_Vertical, symbol Transistor_BJT:TIP122
- removed R23: 220, Resistor_SMD:R_0603_1608Metric_Pad0.98x0.95mm_HandSolder, symbol Device:R_Small
- removed R24: 6.8k, Resistor_SMD:R_0603_1608Metric_Pad0.98x0.95mm_HandSolder, symbol Device:R
- removed R25: 15k, Resistor_SMD:R_0603_1608Metric_Pad0.98x0.95mm_HandSolder, symbol Device:R
- removed R26: 10k, Resistor_SMD:R_0603_1608Metric_Pad0.98x0.95mm_HandSolder, symbol Device:R
- removed R27: 2.7k, Resistor_SMD:R_0603_1608Metric_Pad0.98x0.95mm_HandSolder, symbol Device:R_Small
- removed R33: 100k, Resistor_SMD:R_0603_1608Metric_Pad0.98x0.95mm_HandSolder, symbol Device:R_Small
- removed R36: 1k, Resistor_SMD:R_0603_1608Metric_Pad0.98x0.95mm_HandSolder, symbol Device:R_Small
- removed R37: 330, Resistor_SMD:R_0603_1608Metric_Pad0.98x0.95mm_HandSolder, symbol Device:R_Small
- removed R38: 3, Resistor_SMD:R_1812_4532Metric, symbol Device:R_Small
- removed T3: MABACT0039, Library:MABACT0039_MCM, symbol 2025-03-08_23-32-31:MABACT0039
- removed TH1: 10k, Connector_PinHeader_1.27mm:PinHeader_1x02_P1.27mm_Vertical, symbol Device:Thermistor_NTC
- removed U13: PD0409J5050S2HF, RF_Mini-Circuits:Mini-Circuits_DB1627, symbol RF:TCP-2-10X
- removed U2: LM321, Package_TO_SOT_SMD:SOT-23-5, symbol Amplifier_Operational:LM321
- removed X1, X2: TA1862A, Filter:Filter_SAW_Epcos_DCC6C_3x3mm, symbol RF_Filter:B3715
- added C115: 1n, Capacitor_SMD:C_0603_1608Metric_Pad1.08x0.95mm_HandSolder, symbol Device:C_Small
- added D10: SK6812, LED_SMD:LED_SK6812_PLCC4_5.0x5.0mm_P3.2mm, symbol LED:SK6812
- added D9: BAT54WS, Diode_SMD:D_SOD-323F, symbol Diode:1N4148W
- added FL2: F5QA737M5M2QN-J, SMD5_SAW-B7520_QUA, symbol 2026-07-18_17-48-16:F5QA737M5M2QN-J
- added FL3: FAR-F5KY-740M00-B4UR-Z, FAR-F5KY:FAR-F5KY, symbol F5QA737M5M2QN-J:FAR-F5KY-740M00-B4UR-Z
- added FL4, FL5: B39242B7520P810, SMD5_SAW-B7520_QUA, symbol 2026-07-18_17-48-16:B39242B7520P810
- added HY1: PD0409J5050S2HF, PD0409J5050S2HF, symbol PD0409J5050S2HF:PD0409J5050S2HF
- added Q7: BC847BDW1, Package_TO_SOT_SMD:SOT-363_SC-70-6, symbol Transistor_BJT:BC847BDW1
- added R18, R20: 0, Resistor_SMD:R_0603_1608Metric_Pad0.98x0.95mm_HandSolder, symbol Device:R_Small
- C105: Voltage 35V -> 50V
- C110, C99: footprint Capacitor_SMD:C_0805_2012Metric_Pad1.18x1.45mm_HandSolder -> Capacitor_SMD:C_1206_3216Metric
- C112: footprint Capacitor_SMD:C_0805_2012Metric_Pad1.18x1.45mm_HandSolder -> Capacitor_SMD:C_1206_3216Metric_Pad1.33x1.80mm_HandSolder; Voltage 25V -> 35V
- C13: value 8p2 -> 8.2p
- C16: Voltage 50V -> 35V
- C3, C4: footprint Capacitor_SMD:C_0805_2012Metric_Pad1.18x1.45mm_HandSolder -> Capacitor_SMD:C_0603_1608Metric_Pad1.08x0.95mm_HandSolder
- C36: value 100 -> 470; Voltage 16V -> 35V
- C37: value 100 -> 0; Voltage 16V -> 35V
- C41: value 100n -> 0; Voltage 16V -> 35V
- C51: value 1.8 -> 2.2
- C55: value 100n -> 1n
- C56: value 12 -> 27
- C59: value 4.7 -> 5.6
- C8: Voltage 35V -> 16V
- C9: Voltage 16V -> 35V
- C96: footprint Capacitor_SMD:C_0805_2012Metric_Pad1.18x1.45mm_HandSolder -> Capacitor_SMD:C_1206_3216Metric; Voltage 16V -> 35V
- J2, J4: footprint Connector_Coaxial:SMA_Wurth_60312102114405_Vertical -> Connector_Coaxial:SMA_Amphenol_132289_EdgeMount
- J5: footprint Connector_Coaxial:SMA_Wurth_60312102114405_Vertical -> F_conn:222131
- JP3: value SolderJumper_2_Open -> ds1; footprint Jumper:SolderJumper-2_P1.3mm_Bridged_RoundedPad1.0x1.5mm -> (none)
- JP5: value SolderJumper_2_Open -> ds2; footprint Jumper:SolderJumper-2_P1.3mm_Bridged_RoundedPad1.0x1.5mm -> (none)
- L10: footprint Inductor_SMD:L_0603_1608Metric_Pad1.05x0.95mm_HandSolder -> Inductor_SMD:L_1008_2520Metric_Pad1.43x2.20mm_HandSolder
- L12: footprint Inductor_SMD:L_Walsin_WLFM201209x -> Inductor_SMD:L_0603_1608Metric_Pad1.05x0.95mm_HandSolder
- L4, L5: footprint Inductor_SMD:L_0402_1005Metric -> Inductor_SMD:L_0603_1608Metric_Pad1.05x0.95mm_HandSolder
- L7: value 120n -> 68n
- L8: value 10n -> 12n
- L9: value 180n -> 100n
- R12: footprint Resistor_THT:R_Axial_DIN0614_L14.3mm_D5.7mm_P15.24mm_Horizontal -> res_3550:RES_3550_TEC
- R41, R43, R46, R49: value 270 -> 910
- R42, R47: value 18 -> 5.6
- RV2: footprint Potentiometer_SMD:Potentiometer_Bourns_3269W_Vertical -> Potentiometer_SMD:Potentiometer_Bourns_3314J_Vertical
- U3: value SKY66292-11 -> SKY66312-11
Connections:
- net +13V: no longer JP5.2 (B)
- net +5V: now also D9.2 (A)
- net +9V: no longer C41.1
- net GND: now also C36.2, C41.1, C83.2, D10.1 (VSS), FL2.2 (GND), FL2.3 (GND), FL2.5 (GND), FL3.2 (GND), FL3.5 (GND), FL4.2 (GND), FL4.3 (GND), FL4.5 (GND), FL5.2 (GND), FL5.3 (GND), FL5.5 (GND), HY1.1, HY1.3, HY1.5, Q7.1 (E1), Q7.4 (E2); no longer C41.2, C83.1
- net RFFC_ENX: now also U1.12 (PA10)
- net RFFC_SCLK: now also U1.11 (PA9)
- net RFFC_SDATA: now also U1.8 (PA7); no longer JP3.2 (B)
- net VBUS: now also C83.1, JP3.1 (A), JP5.2 (B); no longer C74.2, C83.2, C87.2, IC2.10 (VDS1), IC2.11 (N/C), IC2.16 (VDS2_2), IC2.17 (N/C), IC2.18 (N/C), IC2.9 (N/C)
- net /PA_ENABLE: now also Q7.3 (C2)
- net at L7.1: now also JP6.3 (B); no longer JP6.1 (A)
- net at C51.2: now also FL2.1 (IN)
- net at Q6.3 (D), R50.1: now also R18.2, R20.1; no longer RV3.1, RV4.3
- net at C5.1, R1.2, R2.1: now also Q7.5 (B2)
- net at J2.1 (In), R1.1: now also C10.1
- net at JP5.1 (A): now also C87.2, IC2.16 (VDS2_2), IC2.17 (N/C), IC2.18 (N/C)
- net at IC1.13 (MIX1_IPN): now also FL3.4 (OUT)
- net at IC1.14 (MIX1_IPP): now also FL3.3 (OUT)
- net at JP1.3 (B), R28.1: now also HY1.6
- net at JP2.3 (B), R28.2: now also HY1.4
- net at C37.1: now also L2.1, L3.1
- net at JP1.1 (A): now also JP6.1 (A); no longer JP6.3 (B)
- net at R41.2, R42.1: now also FL5.4 (OUT)
- net at JP2.2 (C): now also FL3.1 (IN); no longer C36.2
- net at R16.2, U1.3 (PC15): now also D10.2 (DIN)
- net at L10.2, L11.1: now also C41.2
- net at JP4.2 (C): now also FL2.4 (OUT)
- net at L13.1, L2.2: now also C36.1
- net at JP4.3 (B): now also HY1.2
- net at JP7.1 (A): now also C115.1; no longer L9.2
- net at R31.2, R35.2: now also FL4.1 (IN)
- net at R4.2, R5.1: now also Q7.2 (B1)
- net at R6.2, R7.2: now also Q7.6 (C1)
- new net: C74.2, IC2.10 (VDS1), IC2.11 (N/C), IC2.9 (N/C), JP3.2 (B)
- new net: FL4.4 (OUT), FL5.1 (IN)
- new net: R20.2, RV4.3
- new net: R18.1, RV3.1
- new net: C115.2, L9.2
- new net: D10.3 (VDD), D9.1 (K)
Other:
- note added: "*"
- note added: "125MHz 3rd ord. Cheb. 33/75ohm -42dB @740MHz"
- note added: "600MHz 50/75ohm -1dB @740MHz"
- note added: "REF ADJ"
- note added: "TX ATT"
- note added: "±0.25ppm"
- note removed: "125MHz 3rd ord. Cheb. 137/75ohm -42dB @740MHz"
- note removed: "25MHz ±0.25ppm pull ±3ppm Vc=1.65V ±1.15V -151dBc/Hz @10kHz"
- note removed: "5.5V"
- note removed: "6.5V"
- note removed: "700MHz 50/75ohm -2.5dB @740MHz"
- note removed: "ERR AMP"
- note removed: "HEATER"
- note removed: "LIMITER"
- note removed: "OVEN"
- note removed: "x29 725M x30 750M x31 775M"
- company: PZK, SQ5NRY -> PZK
- moved on the sheet: C1, C10, C100, C101, C102, C104, C105, C106, C107, C108, C109, C11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
